File: Kicad/1008-DispDrv/1008.disp2.sch (KiCad schematic (older format))
At the start: 10 parts, among them U301 PCA9655E, U302 NTJD5121N, U303 NTJD5121N, U304 NTJD5121N, U305 NTJD5121N, U306 NTJD5121N, U307 NTJD5121N, U308 NTJD5121N

Commit message: Added part numbers to schematic.  Generated BOM for project.  Created spreadsheet file to total cost of project.
Parts:
- DSP301, DSP302: PartNum (none) -> DISCH1x1
- U301: PartNum (none) -> CHPPCA9655E
- U302, U303, U304, U305, U306, U307, U308: PartNum (none) -> FET2N60V295.m1.60O
Changed lines of the file:
@@
-EESchema Schematic File Version 2  date 12/3/2012 4:24:21 PM
+EESchema Schematic File Version 2  date 12/5/2012 11:19:56 AM
 LIBS:commonpart
 LIBS:power
@@
 Sheet 3 5
 Title "Display Driver"
-Date "3 dec 2012"
+Date "5 dec 2012"
 Rev "A"
 Comp "Open Pinball Project"
@@
 F 0 "U301" H 2900 4350 60  0000 C CNN
 F 1 "PCA9655E" H 2850 4200 60  0000 C CNN
+F 4 "CHPPCA9655E" H 2900 3550 60  0001 C CNN "PartNum"
 	1    2900 3550
 	1    0    0    -1
@@
 F 0 "DSP301" H 10400 2800 60  0000 C CNN
 F 1 "7SEGDISP" H 10400 1800 60  0000 C CNN
+F 4 "DISCH1x1" H 10400 2250 60  0001 C CNN "PartNum"
 	1    10400 2250
 	1    0    0    -1
@@
 F 0 "U303" H 6000 3575 60  0000 C CNN
 F 1 "NTJD5121N" H 5975 3475 60  0000 C CNN
+F 4 "FET2N60V295.m1.60O" H 6350 3200 60  0001 C CNN "PartNum"
 	1    6350 3200
 	1    0    0    -1
@@
 F 0 "U302" H 7200 3575 60  0000 C CNN
 F 1 "NTJD5121N" H 7175 3475 60  0000 C CNN
+F 4 "FET2N60V295.m1.60O" H 7550 3200 60  0001 C CNN "PartNum"
 	2    7550 3200
 	1    0    0    -1
@@
 F 0 "U304" H 8400 3575 60  0000 C CNN
 F 1 "NTJD5121N" H 8375 3475 60  0000 C CNN
+F 4 "FET2N60V295.m1.60O" H 8750 3200 60  0001 C CNN "PartNum"
 	2    8750 3200
 	1    0    0    -1
@@
 F 0 "U302" H 8000 1775 60  0000 C CNN
 F 1 "NTJD5121N" H 7975 1675 60  0000 C CNN
+F 4 "FET2N60V295.m1.60O" H 8350 1400 60  0001 C CNN "PartNum"
 	1    8350 1400
 	1    0    0    -1
@@
 F 0 "U305" H 7000 1775 60  0000 C CNN
 F 1 "NTJD5121N" H 6975 1675 60  0000 C CNN
+F 4 "FET2N60V295.m1.60O" H 7350 1400 60  0001 C CNN "PartNum"
 	1    7350 1400
 	1    0    0    -1
@@
 F 0 "U304" H 6000 1775 60  0000 C CNN
 F 1 "NTJD5121N" H 5975 1675 60  0000 C CNN
+F 4 "FET2N60V295.m1.60O" H 6350 1400 60  0001 C CNN "PartNum"
 	1    6350 1400
 	1    0    0    -1
@@
 F 0 "U303" H 5000 1775 60  0000 C CNN
 F 1 "NTJD5121N" H 4975 1675 60  0000 C CNN
+F 4 "FET2N60V295.m1.60O" H 5350 1400 60  0001 C CNN "PartNum"
 	2    5350 1400
 	1    0    0    -1
@@
 F 0 "U307" H 5000 4975 60  0000 C CNN
 F 1 "NTJD5121N" H 4975 4875 60  0000 C CNN
+F 4 "FET2N60V295.m1.60O" H 5350 4600 60  0001 C CNN "PartNum"
 	2    5350 4600
 	1    0    0    -1
@@
 F 0 "U308" H 6000 4975 60  0000 C CNN
 F 1 "NTJD5121N" H 5975 4875 60  0000 C CNN
+F 4 "FET2N60V295.m1.60O" H 6350 4600 60  0001 C CNN "PartNum"
 	1    6350 4600
 	1    0    0    -1
@@
 F 0 "U305" H 7000 4975 60  0000 C CNN
 F 1 "NTJD5121N" H 6975 4875 60  0000 C CNN
+F 4 "FET2N60V295.m1.60O" H 7350 4600 60  0001 C CNN "PartNum"
 	2    7350 4600
 	1    0    0    -1
@@
 F 0 "U306" H 8000 4975 60  0000 C CNN
 F 1 "NTJD5121N" H 7975 4875 60  0000 C CNN
+F 4 "FET2N60V295.m1.60O" H 8350 4600 60  0001 C CNN "PartNum"
 	1    8350 4600
 	1    0    0    -1
@@
 F 0 "U308" H 8400 6775 60  0000 C CNN
 F 1 "NTJD5121N" H 8375 6675 60  0000 C CNN
+F 4 "FET2N60V295.m1.60O" H 8750 6400 60  0001 C CNN "PartNum"
 	2    8750 6400
 	1    0    0    -1
@@
 F 0 "U306" H 7200 6775 60  0000 C CNN
 F 1 "NTJD5121N" H 7175 6675 60  0000 C CNN
+F 4 "FET2N60V295.m1.60O" H 7550 6400 60  0001 C CNN "PartNum"
 	2    7550 6400
 	1    0    0    -1
@@
 F 0 "U307" H 6000 6775 60  0000 C CNN
 F 1 "NTJD5121N" H 5975 6675 60  0000 C CNN
+F 4 "FET2N60V295.m1.60O" H 6350 6400 60  0001 C CNN "PartNum"
 	1    6350 6400
 	1    0    0    -1
@@
 F 0 "DSP302" H 10400 6000 60  0000 C CNN
 F 1 "7SEGDISP" H 10400 5000 60  0000 C CNN
+F 4 "DISCH1x1" H 10400 5450 60  0001 C CNN "PartNum"
 	1    10400 5450
 	1    0    0    -1
