File: Kicad/1008-DispDrv/1008.disp3.sch (KiCad schematic (older format))
At the start: 10 parts, among them U201 PCA9655E, U202 NTJD5121N, U203 NTJD5121N, U204 NTJD5121N, U205 NTJD5121N, U206 NTJD5121N, U207 NTJD5121N, U208 NTJD5121N

Commit message: Added silkscreen for cutouts for connectors.  Added connectors for distributing VDD.  Move connectors closer to the edge.  Add more clearance for mounting hardware.  Change connectors to right angle because of height restrictions.
Changed lines of the file:
@@
-EESchema Schematic File Version 2  date 11/18/2012 8:37:23 PM
+EESchema Schematic File Version 2  date 11/27/2012 11:36:53 AM
 LIBS:commonpart
 LIBS:power
@@
 Sheet 2 5
 Title "Display Driver"
-Date "19 nov 2012"
+Date "27 nov 2012"
 Rev "A"
 Comp "Open Pinball Project"
@@
 Connection ~ 7800 4000
 Wire Wire Line
-	7800 4000 7800 5800
+	7800 5800 7800 4000
 Connection ~ 7450 4000
 Wire Wire Line
@@
 Connection ~ 6800 800
 Wire Wire Line
-	6800 800  6800 2400
+	6800 2400 6800 800
 Connection ~ 8450 800
 Wire Wire Line
-	8850 800  8850 2700
+	8850 2700 8850 800
 Wire Wire Line
 	8850 800  5450 800
@@
 	11100 2300 11000 2300
 Wire Wire Line
-	9700 2500 9800 2500
-Wire Wire Line
-	9700 2700 9700 2500
+	9800 2500 9700 2500
+Wire Wire Line
+	9700 2500 9700 2700
 Wire Wire Line
 	7450 1900 7450 2100
@@
 	9700 5700 9800 5700
 Wire Wire Line
-	11100 5500 11000 5500
+	11000 5500 11100 5500
 Connection ~ 11100 5700
 Wire Wire Line
@@
 Connection ~ 11100 5600
 Wire Wire Line
-	11100 5900 11100 5500
+	11100 5500 11100 5900
 Connection ~ 11100 5800
 Wire Wire Line

Commit message: Added part numbers to schematic.  Generated BOM for project.  Created spreadsheet file to total cost of project.
Parts:
- DSP201, DSP202: PartNum (none) -> DISCH1x1
- U201: PartNum (none) -> CHPPCA9655E
- U202, U203, U204, U205, U206, U207, U208: PartNum (none) -> FET2N60V295.m1.60O
Changed lines of the file:
@@
-EESchema Schematic File Version 2  date 12/3/2012 4:24:21 PM
+EESchema Schematic File Version 2  date 12/5/2012 11:19:56 AM
 LIBS:commonpart
 LIBS:power
@@
 Sheet 2 5
 Title "Display Driver"
-Date "3 dec 2012"
+Date "5 dec 2012"
 Rev "A"
 Comp "Open Pinball Project"
@@
 F 0 "U201" H 2900 4350 60  0000 C CNN
 F 1 "PCA9655E" H 2850 4200 60  0000 C CNN
+F 4 "CHPPCA9655E" H 2900 3550 60  0001 C CNN "PartNum"
 	1    2900 3550
 	1    0    0    -1
@@
 F 0 "DSP201" H 10400 2800 60  0000 C CNN
 F 1 "7SEGDISP" H 10400 1800 60  0000 C CNN
+F 4 "DISCH1x1" H 10400 2250 60  0001 C CNN "PartNum"
 	1    10400 2250
 	1    0    0    -1
@@
 F 0 "U203" H 6000 3575 60  0000 C CNN
 F 1 "NTJD5121N" H 5975 3475 60  0000 C CNN
+F 4 "FET2N60V295.m1.60O" H 6350 3200 60  0001 C CNN "PartNum"
 	1    6350 3200
 	1    0    0    -1
@@
 F 0 "U202" H 7200 3575 60  0000 C CNN
 F 1 "NTJD5121N" H 7175 3475 60  0000 C CNN
+F 4 "FET2N60V295.m1.60O" H 7550 3200 60  0001 C CNN "PartNum"
 	2    7550 3200
 	1    0    0    -1
@@
 F 0 "U204" H 8400 3575 60  0000 C CNN
 F 1 "NTJD5121N" H 8375 3475 60  0000 C CNN
+F 4 "FET2N60V295.m1.60O" H 8750 3200 60  0001 C CNN "PartNum"
 	2    8750 3200
 	1    0    0    -1
@@
 F 0 "U202" H 8000 1775 60  0000 C CNN
 F 1 "NTJD5121N" H 7975 1675 60  0000 C CNN
+F 4 "FET2N60V295.m1.60O" H 8350 1400 60  0001 C CNN "PartNum"
 	1    8350 1400
 	1    0    0    -1
@@
 F 0 "U205" H 7000 1775 60  0000 C CNN
 F 1 "NTJD5121N" H 6975 1675 60  0000 C CNN
+F 4 "FET2N60V295.m1.60O" H 7350 1400 60  0001 C CNN "PartNum"
 	1    7350 1400
 	1    0    0    -1
@@
 F 0 "U204" H 6000 1775 60  0000 C CNN
 F 1 "NTJD5121N" H 5975 1675 60  0000 C CNN
+F 4 "FET2N60V295.m1.60O" H 6350 1400 60  0001 C CNN "PartNum"
 	1    6350 1400
 	1    0    0    -1
@@
 F 0 "U203" H 5000 1775 60  0000 C CNN
 F 1 "NTJD5121N" H 4975 1675 60  0000 C CNN
+F 4 "FET2N60V295.m1.60O" H 5350 1400 60  0001 C CNN "PartNum"
 	2    5350 1400
 	1    0    0    -1
@@
 F 0 "U207" H 5000 4975 60  0000 C CNN
 F 1 "NTJD5121N" H 4975 4875 60  0000 C CNN
+F 4 "FET2N60V295.m1.60O" H 5350 4600 60  0001 C CNN "PartNum"
 	2    5350 4600
 	1    0    0    -1
@@
 F 0 "U208" H 6000 4975 60  0000 C CNN
 F 1 "NTJD5121N" H 5975 4875 60  0000 C CNN
+F 4 "FET2N60V295.m1.60O" H 6350 4600 60  0001 C CNN "PartNum"
 	1    6350 4600
 	1    0    0    -1
@@
 F 0 "U205" H 7000 4975 60  0000 C CNN
 F 1 "NTJD5121N" H 6975 4875 60  0000 C CNN
+F 4 "FET2N60V295.m1.60O" H 7350 4600 60  0001 C CNN "PartNum"
 	2    7350 4600
 	1    0    0    -1
@@
 F 0 "U206" H 8000 4975 60  0000 C CNN
 F 1 "NTJD5121N" H 7975 4875 60  0000 C CNN
+F 4 "FET2N60V295.m1.60O" H 8350 4600 60  0001 C CNN "PartNum"
 	1    8350 4600
 	1    0    0    -1
@@
 F 0 "U208" H 8400 6775 60  0000 C CNN
 F 1 "NTJD5121N" H 8375 6675 60  0000 C CNN
+F 4 "FET2N60V295.m1.60O" H 8750 6400 60  0001 C CNN "PartNum"
 	2    8750 6400
 	1    0    0    -1
@@
 F 0 "U206" H 7200 6775 60  0000 C CNN
 F 1 "NTJD5121N" H 7175 6675 60  0000 C CNN
+F 4 "FET2N60V295.m1.60O" H 7550 6400 60  0001 C CNN "PartNum"
 	2    7550 6400
 	1    0    0    -1
@@
 F 0 "U207" H 6000 6775 60  0000 C CNN
 F 1 "NTJD5121N" H 5975 6675 60  0000 C CNN
+F 4 "FET2N60V295.m1.60O" H 6350 6400 60  0001 C CNN "PartNum"
 	1    6350 6400
 	1    0    0    -1
@@
 F 0 "DSP202" H 10400 6000 60  0000 C CNN
 F 1 "7SEGDISP" H 10400 5000 60  0000 C CNN
+F 4 "DISCH1x1" H 10400 5450 60  0001 C CNN "PartNum"
 	1    10400 5450
 	1    0    0    -1
